File: MiniVersion/MiniVersion.kicad_pcb (KiCad board)
At the start: 2 copper layers, 38.6 x 27 mm, 24 parts, among them J1 PowerIn, J2 Conn_01x03, J3 Conn_01x03, J4 Program, U2 LTV-355T, U3 VTX-214-003-203, U4 ESP-12E

Commit message: update
Parts:
- moved U2 0.60 mm to (142.4, 78.0)
Routing:
- net Net-(D2-A): track 10.0 -> 9.37 mm
- net GND: track 2.34 -> 2.94 mm
Other:
- board size 38.6 x 27 mm -> 56 x 27 mm
